Commit message: 8-21_1

File: src/agrobot_description/urdf/robot_display.urdf (robot description, URDF)
Before this commit: robot robot, 7 links, 6 joints
Links:
- removed link laser_link
- added link liser_link, mass 0.1; collision cylinder length=0.02 radius=0.02; visual cylinder length=0.02 radius=0.02
Joints:
- joint laser_joint: child laser_link -> liser_link

Commit message: 9-6_1

File: src/agrobot_description/urdf/robot_display.urdf (robot description, URDF)
Before this commit: robot robot, 7 links, 6 joints
Links:
- added link depth_camera_link, mass 0.1; collision box size=0.1 0.1 0.05; visual box size=0.1 0.1 0.05
Joints:
- added joint depth_camera_joint: type fixed, parent base_link, child depth_camera_link, origin xyz=0.1 0 0.1 rpy=0 0 0
