Commit message: 9-10_1

File: src/agrobot_description/urdf/robot_camera_display.urdf (robot description, URDF)
Before this commit: robot robot, 7 links, 6 joints
Links:
- added link depth_camera_link, mass 0.1; collision box size=0.05 0.1 0.03; visual box size=0.05 0.1 0.03
- added link link_camera_fake
Joints:
- added joint depth_camera_joint: type fixed, parent base_link, child depth_camera_link, origin xyz=0.1 0 0.6 rpy=0 0 0
- added joint joint_camera_fake: type fixed, parent depth_camera_link, child link_camera_fake, origin xyz=0 0 0 rpy=-1.5708 0 -1.5708
